File: Sport Analyzer 1.0.1/Sport Analyzer 1.0.1.brd (EAGLE design)
At the start: 122.7 x 68.6 mm, 26 parts, among them IC2 7805DT, Q1 MMBT4403, U1 HX711

Commit message: SP 1.0.1 PMMA case 1
Routing:
- net N$42: track 10.6 -> 9.41 mm
Other:
- board text added: "Sport Analyzer"
- board text added: "by Xavier Cano-Ferrer"
- board text removed: "Sport Analyzer 1.0"
Changed lines of the file:
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@@
 <hole x="82.55" y="61.83" drill="3"/>
 <hole x="6.25" y="4.21" drill="3"/>
-<text x="104.41" y="20.49" size="1.6764" layer="25" rot="R90">Sport Analyzer 1.0</text>
-<hole x="113.94" y="44.53" drill="2"/>
-<hole x="91.73" y="31.26" drill="2"/>
-<hole x="114.16" y="17.3" drill="2"/>
+<text x="103.41" y="9.49" size="1.6764" layer="25" rot="R90">Sport Analyzer</text>
+<hole x="91.65" y="44.26" drill="2"/>
+<hole x="114.02" y="30.8" drill="2"/>
+<hole x="91.66" y="17.28" drill="2"/>
+<text x="107.41" y="9.49" size="1.6764" layer="25" rot="R90">by Xavier Cano-Ferrer</text>
 </plain>
 <attributes>
@@
 </element>
 <element name="IC2" library="linear" library_urn="urn:adsk.eagle:library:262" package="TO252" package3d_urn="urn:adsk.eagle:package:16415/2" value="7805DT" x="22.86" y="46.99" smashed="yes" rot="R90">
-<attribute name="NAME" x="25.4" y="43.18" size="1.27" layer="25" rot="R180"/>
+<attribute name="NAME" x="22.89" y="43.37" size="1.27" layer="25" rot="R180"/>
 <attribute name="POPULARITY" value="0" x="22.86" y="46.99" size="1.778" layer="27" rot="R90" display="off"/>
 <attribute name="VALUE" x="25.4" y="52.07" size="1.27" layer="27" rot="R180"/>
 </element>
 <element name="C8" library="SparkFun-Capacitors" package="0603-CAP" value="0.33uF" x="31.29" y="43.05" smashed="yes" rot="R180">
-<attribute name="NAME" x="32.179" y="42.288" size="0.4064" layer="25" font="vector" rot="R180"/>
+<attribute name="NAME" x="31.739" y="46.118" size="0.8128" layer="25" font="vector" rot="R180"/>
 <attribute name="PROD_ID" value="CAP-08604" x="31.29" y="43.05" size="1.778" layer="27" rot="R180" display="off"/>
-<attribute name="VALUE" x="32.306" y="44.193" size="0.4064" layer="27" font="vector" rot="R180"/>
+<attribute name="VALUE" x="33.286" y="45.023" size="0.8128" layer="25" font="vector" rot="R180"/>
 </element>
 <element name="C9" library="SparkFun-Capacitors" package="0603-CAP" value="0.1uF" x="38.44" y="40.05" smashed="yes" rot="R90">
@@
 </element>
 <element name="S2" library="switch" library_urn="urn:adsk.eagle:library:380" package="TL3XPO" package3d_urn="urn:adsk.eagle:package:27745/1" value="TL32PO" x="97.2" y="64.6" smashed="yes" rot="R180">
-<attribute name="NAME" x="104.18" y="61.025" size="1.778" layer="25" rot="R180"/>
+<attribute name="NAME" x="105.98" y="65.015" size="1.778" layer="25" rot="R180"/>
 <attribute name="POPULARITY" value="2" x="108.2" y="53" size="1.778" layer="27" rot="R180" display="off"/>
-<attribute name="VALUE" x="112.08" y="65.68" size="1.778" layer="27" rot="R180"/>
+<attribute name="VALUE" x="110.28" y="61.22" size="1.778" layer="27" rot="R180"/>
 </element>
 <element name="S3" library="switch-omron" library_urn="urn:adsk.eagle:library:377" package="B3F-10XX" package3d_urn="urn:adsk.eagle:package:27496/1" value="" x="34.98" y="62.29" smashed="yes">
@@
 <contactref element="S2" pad="1"/>
 <contactref element="BT1" pad="+"/>
-<wire x1="99.74" y1="64.6" x2="99.74" y2="57.94" width="0.8128" layer="1"/>
-<wire x1="98.37" y1="56.57" x2="96.41" y2="56.57" width="0.8128" layer="1"/>
-<wire x1="99.74" y1="57.94" x2="98.37" y2="56.57" width="0.8128" layer="1"/>
+<wire x1="96.41" y1="56.57" x2="99.74" y2="59.9" width="0.8128" layer="1"/>
+<wire x1="99.74" y1="59.9" x2="99.74" y2="64.6" width="0.8128" layer="1"/>
 </signal>
 <signal name="N$9">
