File: Teensy 4 version/Design files/Sport Analyzer Teensy4 (Mosfets).brd (EAGLE design)
At the start: 122.7 x 68.6 mm, 27 parts, among them IC2 7805DT, Q1 MMBT4403, U1 HX711, U2 TXB0108PWR

Commit message: Teensy 4 logic level shifters V2
Parts:
- removed U2: TXB0108PWR, microbuilder:TSSOP20
- added Q2, Q3, Q4: BSS138, SparkFun:SOT23-3
- added R10, R11, R6, R7, R8, R9: 10K, SparkFun:0603-RES
Connections:
- net CLK: now also U$2.13-SCK/CRX1/LED
- net ENC_A: now also Q2.3, R7.2; no longer U2.20
- net ENC_A_3V3: now also Q2.2, R6.2; no longer U2.1
- net ENC_B: now also Q3.3, R9.2; no longer U2.18
- net ENC_B_3V3: now also Q3.2, R8.2; no longer U2.3
- net ENC_Z: now also Q4.3, R11.2; no longer U2.17
- net ENC_Z_3V3: now also Q4.2, R10.2; no longer U2.4
- net GND: no longer U2.11
- net VCC: now also R11.1, R7.1, R9.1; no longer U2.19
- net VDD: now also Q2.1, Q3.1, Q4.1, R10.1, R6.1, R8.1; no longer U2.10, U2.2
Routing:
- net CLK: track 0.00 -> 38.4 mm
- net ENC_Z_3V3: track 28.8 -> 49.7 mm
- net ENC_Z: track 7.86 -> 27.5 mm, vias 0 -> 2
- net ENC_B_3V3: track 29.6 -> 46.0 mm
- net ENC_B: track 5.25 -> 20.5 mm
- net ENC_A_3V3: track 18.9 -> 32.1 mm, vias 1 -> 3
- net VDD: track 118.2 -> 129.8 mm, vias 0 -> 5
- net ENC_A: track 7.96 -> 18.4 mm
- net GND: track 178.9 -> 189.2 mm
- net VCC: track 194.3 -> 197.2 mm
- net 9V: track 237.3 -> 236.7 mm
