File: Chronojump version/Teensy 3.2 version/Design files/Sport Analyzer Chronojump.sch (EAGLE design)
At the start: 35 parts, among them IC2 7805DT, Q1 MMBT4403, Q2 BSS138, Q3 BSS138, Q4 BSS138, U1 HX711

Commit message: Teensy 4 update
Parts:
- removed LOAD_CELL: RJ11-2L-B, con-tycoelectronics:RJ11-2L-B
- removed Q2, Q3, Q4: BSS138, SparkFun:MOSFET-NCHANNELSMD
- removed R10, R11, R6, R7, R8, R9: 10K, SparkFun:RESISTOR0603-RES
- removed U$2: TEENSY40, teensy:TEENSY40
- added A+, A-, AVDD, GND: (no value), wirepad_xavi:3,81/1,4
- added CP_TRIG: RC-5231, con-lumberg:RC-5231
- added D1: (no value), adafruit:DIODESOD-123
- added U$1: TEENSY_3.1-3.2_DIL, Teensy_3_and_LC_Series_Boards_v1.4:TEENSY_3.1-3.2_DIL
- ENCODER: value RJ11-2L-B -> RJ45-8PTH; device con-tycoelectronics:RJ11-2L-B -> SparkFun:RJ45-8PTH
Connections:
- removed net ENC_A_3V3: Q2.S, R6.2, U$2.8-IN1/TX2
- removed net ENC_B_3V3: Q3.S, R8.2, U$2.9-OUT1C
- removed net ENC_Z: ENCODER.4, Q4.D, R11.2
- removed net ENC_Z_3V3: Q4.S, R10.2, U$2.7-OUT1A/RX2
- new net 9VD: C8.1, D1.C, IC2.VI
- new net CP_TRIG: CP_TRIG.T, U$1.16/A2/T
- net 9V: now also D1.A; no longer C8.1, IC2.VI
- net A+: now also A+.P; no longer LOAD_CELL.3
- net A-: now also A-.P; no longer LOAD_CELL.4
- net AVDD: now also AVDD.P; no longer LOAD_CELL.6
- net CLK: now also U$1.14/A1; no longer U$2.13-SCK/CRX1/LED
- net CS: now also U$1.21/A7/PWM; no longer U$2.10-CS
- net D/C: now also U$1.20/A6/PWM; no longer U$2.20-A6/TX5/LRCLK1
- net DAT: now also U$1.2; no longer U$2.2-OUT2
- net ENC_A: now also ENCODER.3, U$1.8/TX3; no longer ENCODER.6, Q2.D, R7.2
- net ENC_B: now also ENCODER.1, U$1.9/RX2/PWM; no longer ENCODER.5, Q3.D, R9.2
- net GND: now also CP_TRIG.S, ENCODER.7, GND.P, U$1.GND; no longer ENCODER.1, ENCODER.2, LOAD_CELL.2, LOAD_CELL.5, U$2.GND1, U$2.GND2, U$2.GND3
- net MISO: now also U$1.12/MISO; no longer U$2.12-MISO/MQSL
- net MOSI: now also U$1.7/RX3; no longer U$2.11-MOSI/CTX1
- net N$8: now also U$1.4/CAN-RX/PWM; no longer U$2.4-BCLK1
- net N$9: now also U$1.5/PWM; no longer U$2.5-IN2
- net SCK: now also U$1.3/CAN-TX/PWM; no longer U$2.3-LRCLK2
- net SD_CS: now also U$1.6/PWM; no longer U$2.6-OUT1D
- net VCC: now also ENCODER.8, TFT_2.8"_RIGHT.2, U$1.VIN; no longer ENCODER.3, R11.1, R7.1, R9.1, U$2.VIN
- net VDD: now also U$1.3.3V; no longer Q2.G, Q3.G, Q4.G, R10.1, R6.1, R8.1, TFT_2.8"_RIGHT.2, U$2.3V3-1, U$2.3V3-2
Other:
- note added: "Coaxial connector"
- note added: "Encoder"
- note added: "Load cell"
- note removed: "Load cell 24bit ADC"
- note removed: "Logic level shifter"
- note removed: "Teensy 4.0"
- moved on the sheet: BT1, C1, C2, C3, C5, C6, C7, C8, C9, IC2, L1, Q1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
