File: Chronojump version/Teensy 4.0 version/Design files/Sport Analyzer Chronojump Teensy 4 (4 buttons).sch (EAGLE design)
At the start: 40 parts, among them IC2 7805DT, Q1 MMBT4403, Q2 BSS138, Q3 BSS138, SW1 C&K_COMPONENTS_D6R40F1LFSC&K_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, SW2 C&K_COMPONENTS_D6R40F1LFSC&K_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, SW3 C&K_COMPONENTS_D6R40F1LFSC&K_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, SW4 C&K_COMPONENTS_D6R40F1LFSC&K_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, U1 HX711

Commit message: RTC DS1302 v1
Parts:
- added Q4: 32.768, microbuilder:CRYSTAL8.0X3.8
- added U$1: DS1302, adafruit:DS1302
Connections:
- removed net N$14: BT2.+, U$2.VBAT
- new net N$18: BT2.+, U$1.VBAT
- new net N$8: Q4.2, U$1.X1
- new net N$9: Q4.1, U$1.X2
- new net RTC_CE: U$1.CE, U$2.7-OUT1A/RX2
- new net RTC_I/O: U$1.I/O, U$2.5-IN2
- new net RTC_SCLK: U$1.SCLK, U$2.4-BCLK1
- net GND: now also U$1.GND
- net VDD: now also U$1.VCC
Other:
- note added: "Real time clock"
- moved on the sheet: BT2
